Commit message: initial commit

File: p3dx_description/urdf/pioneer3dx.xacro (robot description, xacro)
@@ -33,5 +33,5 @@
   <link name="$(arg base_frame)">
     <inertial>
-      <mass value="3.5" />
+      <mass value="26" />
       <!--<origin xyz="-0.025 0 -0.223"/> -->
       <origin xyz="-0.05 0 0" />

Commit message: Amal small changes to params

File: p3dx_description/urdf/pioneer3dx.xacro (robot description, xacro)
@@ -33,5 +33,5 @@
   <link name="$(arg base_frame)">
     <inertial>
-      <mass value="26" />
+      <mass value="25" />
       <!--<origin xyz="-0.025 0 -0.223"/> -->
       <origin xyz="-0.05 0 0" />
